File: PCB/prec_cc_cv_psu.sch (KiCad schematic (older format))
At the start: 64 parts, among them U1 ISL21070, U2 LM358, U3 LM358, U4 LT3080

Commit message: Schematic update
Updated schematic:
- added crystal
- renumerated parts
- quick and dirty fix of labels
Parts:
- added C10, C9: C, symbol C
- added R1: 10K, symbol R
- added SW2: SW_PUSH, symbol SW_PUSH
- added Y1: Crystal, symbol Crystal
- gave numbers to parts that had none: 59
Connections:
- net labels added: RST, RXD, TXD
- wire segments 165 -> 180
